Commit message: Cleaned and polished code

File: urdf/navvis.xacro (robot description, xacro)
@@ -18,53 +18,4 @@
         </collision>
     </link>
-    <!-- child of the base -->
-    <!-- <link name="laser_vert_bottom">
-        <visual>
-            <geometry>
-                <box size="0.062 0.062 .087" />
-            </geometry>
-        </visual>
-        <collision>
-            <geometry>
-                <box size="0.062 0.062 .087" />
-            </geometry>
-        </collision>
-    </link> -->
-    <!-- <link name="laser_vert_top_right">
-        <visual>
-            <geometry>
-                <box size="0.062 0.062 .087" />
-            </geometry>
-        </visual>
-        <collision>
-            <geometry>
-                <box size="0.062 0.062 .087" />
-            </geometry>
-        </collision>
-    </link>-->
-    <!-- <link name="laser_vert_top_left">
-        <visual>
-            <geometry>
-                <box size="0.062 0.062 .087" />
-            </geometry>
-        </visual>
-        <collision>
-            <geometry>
-                <box size="0.062 0.062 .087" />
-            </geometry>
-        </collision>
-    </link> -->
-    <!-- <link name="laser_horiz">
-        <visual>
-            <geometry>
-                <cylinder radius=".052" length=".072"/>
-            </geometry>
-        </visual>
-        <collision>
-            <geometry>
-                <box size="0.062 0.062 .087" />
-            </geometry>
-        </collision>
-    </link> -->
     <!-- Left / Right Wheels -->
     <xacro:macro name="gen_wheel" params="side reflect">
@@ -86,12 +37,10 @@
             <origin xyz="-0.10 ${ reflect * 0.4 } 0.0" rpy="${ pi / -2 } 0.0 0.0" />
             <axis xyz="0 0 1" />
-            <limit effort="1.0" velocity="1.0"/>
             <!-- limit is not required for continuous joints -->
         </joint>
     </xacro:macro>
-    <!-- Create the left and right wheel with xacro -->
     <xacro:gen_wheel side="left" reflect="1" />
     <xacro:gen_wheel side="right" reflect="-1"/>
-    <!-- Create the center wheel -->
+    <!-- Center wheel -->
     <link name="wheel_center">
         <visual>
@@ -111,8 +60,7 @@
         <origin xyz="0.10 0.0 -0.05" rpy="${ pi / -2 } 0.0 0.0" />
         <axis xyz="0 0 1" />
-        <limit effort="1.0" velocity="1.0"/>
         <!-- limit is not required for continuous joints -->
     </joint>
-<!-- JOINTS -->
+    <!-- Laser Vertices -->
     <xacro:include filename="$(find gazebo_plugins)/test/multi_robot_scenario/xacro/laser/hokuyo.xacro" />
     <xacro:laser
@@ -139,23 +87,3 @@
         <origin xyz="0.2325 0.0001 1.9201" rpy="-0.0012 0.1146 -0.0015" />
     </xacro:VLP-16>
-    <!-- <joint name="base_laser_vert_bottom_joint" type="fixed">
-        <parent link="base"/>
-        <child link="laser_vert_bottom" />
-        <origin xyz="0.3158 -0.0021 0.5100" rpy="3.1355 -1.3045 0.0025" />
-    </joint> -->
-    <!-- <joint name="base_laser_horiz_joint" type="fixed">
-        <parent link="base"/>
-        <child link="laser_horiz" />
-        <origin xyz="0.2325 0.0001 1.9201" rpy="-0.0012 0.1146 -0.0015" />
-    </joint> -->
-    <!-- <joint name="base_laser_vert_top_left_joint" type="fixed">
-        <parent link="base"/>
-        <child link="laser_vert_top_left" />
-        <origin xyz="0.2997 0.1531 1.8443" rpy="1.1780 0.6198 1.9560" />
-    </joint>
-    <joint name="base_laser_vert_top_right_joint" type="fixed">
-        <parent link="base"/>
-        <child link="laser_vert_top_right" />
-        <origin xyz="0.2978 -0.1450 1.8451" rpy="-1.760 0.6313 -1.9377" />
-    </joint> -->
 </robot>
